File: USB_3.0_Hub/USB_3.0_Hub.kicad_pcb (KiCad board)
At the start: 2 copper layers, 0 parts

Commit message: push
Parts:
- added SW1: I2C Selector, Button_Switch_SMD:Nidec_Copal_CAS-120A, F.Cu at (111.9, 68.6)
- added U1: TUSB8041, Package_DFN_QFN:QFN-64-1EP_9x9mm_P0.5mm_EP6x6mm_ThermalVias, F.Cu at (67.5, 84.3)
- added U2: AT24CS04-XHM, Package_SO:TSSOP-8_4.4x3mm_P0.65mm, F.Cu at (89.8, 59.7)
- added U3: FT4232H, Package_QFP:LQFP-64-1EP_10x10mm_P0.5mm_EP5x5mm_ThermalVias, F.Cu at (78.2, 64.6)
- added U4: MAX15062A, Package_DFN_QFN:DFN-8_2x2mm_P0.5mm, F.Cu at (116.8, 85.6)
- added U5: ADP2108AUJ-1.1, Package_TO_SOT_SMD:TSOT-23-5, F.Cu at (87.1, 85.9)
- added U6: 93LCxxBxxOT, Package_TO_SOT_SMD:SOT-23-6, F.Cu at (104.9, 86.4)
