File: USB_3.0_Hub/USB_3.0_Hub.kicad_sch (KiCad schematic)
At the start: 16 parts, among them J1 USB_UP, J2 USB_DN1, J3 USB_DN2, J4 USB_DN3, J5 I2C EEPROM, SW1 I2C Selector, U1 TUSB8041, U2 AT24CS04-XHM, Y1 24MHz

Commit message: added stuff
Parts:
- added U3: FT4232H, symbol Interface_USB:FT4232H
Connections:
- net GND1: now also U1.65 (VSS)
- net VDD: now reaches U1.13 (VDD)
- net VDD: now also U1.21 (VDD), U1.28 (VDD), U1.31 (VDD), U1.5 (VDD), U1.51 (VDD), U1.57 (VDD), U1.8 (VDD)
- net VDD33: now reaches U1.16 (VDD33)
- net VDD33: now also U1.34 (VDD33), U1.52 (VDD33), U1.63 (VDD33)
Other:
- note added: "FT4232H JTAG/I2C/SPI"
- note added: "Power Supply"
- note added: "USB 3.0 4-Port Hub"
- moved on the sheet: U1

Commit message: abruh
Parts:
- added C10, C11, C12, C13, C14, C17, C18, C19, C20, C8, C9: 0.1uF, symbol Device:C_Small
- added C15, C21, C6: 10uF, symbol Device:C_Small
- added C16, C3: 20pF, symbol Device:C
- added C4: 1uF, symbol Device:C_Small
- added C5: 10pF, symbol Device:C_Small
- added C7: 4.7uF, symbol Device:C_Small
- added L1: 1uH, symbol Device:L_Small
- added L2: 33uH, symbol Device:L_Small
- added R10, R6, R7, R8, R9: 4k7, symbol Device:R_Small
- added R11: 9.53k/1%, symbol Device:R_Small
- added R12: 90k, symbol Device:R_Small
- added R13, R16: 10k, symbol Device:R_Small
- added R14: 1M, symbol Device:R
- added R15: 2k, symbol Device:R_Small
- added SW2: SW_SPDT, symbol Switch:SW_SPDT
- added U4: MAX15062A, Package_DFN_QFN:DFN-8_2x2mm_P0.5mm, symbol Regulator_Switching:MAX15062A
- added U5: ADP2108AUJ-1.1, Package_TO_SOT_SMD:TSOT-23-5, symbol Regulator_Switching:ADP2108AUJ-1.1
- added U6: 93LCxxBxxOT, Package_TO_SOT_SMD:SOT-23-6, symbol Memory_EEPROM:93LCxxBxxOT
- added Y2: 24MHz, symbol Device:Crystal
- C1, C2: value C -> 18pF
- U3: footprint (none) -> Package_QFP:LQFP-64-1EP_10x10mm_P0.5mm_EP5x5mm_ThermalVias
Connections:
- net VDD33 is gone; now on net +3.3V: U1.16 (VDD33), U1.34 (VDD33), U1.52 (VDD33), U1.63 (VDD33)
- net GND1: now also U3.1 (GND), U3.10 (AGND), U3.11 (GND), U3.13 (TEST), U3.15 (GND), U3.25 (GND), U3.35 (GND), U3.47 (GND), U3.5 (GND), U3.51 (GND), C10.2, C11.2, C12.2, C13.2, C14.2, C15.2, C16.1, C17.2, C18.2, C19.2, C20.2, C21.2, C3.2, C4.2, C5.2, C6.2, C7.2, C8.2, C9.2, R10.1, R11.1, R13.1, R16.2, R6.1, R7.1, R8.1, R9.1, SW2.1 (A), U4.7 (GND), U5.2 (GND), U6.2 (GND)
- net SCL/SMBCLK: no longer U2.6 (SCL)
- net SDA/SMBDAT: no longer U2.5 (SDA)
- net VCORE: now reaches U3.12 (VCORE)
- net VCORE: now also U3.37 (VCORE), U3.64 (VCORE)
- net FT XI: now reaches U3.2 (OSCI)
- net FT XI: now also C16.2, R14.2, Y2.2
- net VIO: now reaches U3.20 (VCCIO)
- net VIO: now also U3.31 (VCCIO), U3.42 (VCCIO), U3.56 (VCCIO)
- net FT XO: now reaches U3.3 (OSCO)
- net FT XO: now also C3.1, R14.1, Y2.1
- net VPHY: now reaches U3.4 (VPHY)
- net FTDATA: now reaches U3.61 (EEDATA)
- net FTDATA: now also R15.1, U6.3 (DI)
- net FTCLK: now reaches U3.62 (EECLK)
- net FTCLK: now also U6.4 (CLK)
- net FTCS: now reaches U3.63 (EECS)
- net FTCS: now also U6.5 (CS)
- net FT D-: now reaches U3.7 (DM)
- net FT D+: now reaches U3.8 (DP)
- net VPLL: now reaches U3.9 (VPLL)
- net +3.3V: now reaches U2.8 (VCC)
- net +3.3V: now also C17.1, C18.1, C19.1, C20.1, C21.1, C6.1, C7.1, L2.2, SW2.3 (C), U4.4 (FB/Vout), U5.1 (Vin), U5.3 (EN), U6.6 (VCC)
- net USB_DP_DN1: now reaches U1.1 (USB_DP_DN1)
- net USB_DM_DN2: now reaches U1.10 (USB_DM_DN2)
- net USB_SSTXP_DN2: now reaches U1.11 (USB_SSTXP_DN2)
- net USB_SSTXM_DN2: now reaches U1.12 (USB_SSTXM_DN2)
- net USB_SSRXP_DN2: now reaches U1.14 (USB_SSRXP_DN2)
- net USB_SSRXM_DN2: now reaches U1.15 (USB_SSRXM_DN2)
- net USB_DP_DN3: now reaches U1.17 (USB_DP_DN3)
- net USB_DM_DN3: now reaches U1.18 (USB_DM_DN3)
- net USB_SSTXP_DN3: now reaches U1.19 (USB_SSTXP_DN3)
- net USB_DM_DN1: now reaches U1.2 (USB_DM_DN1)
- net USB_SSTXM_DN3: now reaches U1.20 (USB_SSTXM_DN3)
- net USB_SSRXP_DN3: now reaches U1.22 (USB_SSRXP_DN3)
- net USB_SSRXM_DN3: now reaches U1.23 (USB_SSRXM_DN3)
- net USB_DP_DN4: now reaches U1.24 (USB_DP_DN4)
- net USB_DM_DN4: now reaches U1.25 (USB_DM_DN4)
- net USB_SSTXP_DN4: now reaches U1.26 (USB_SSTXP_DN4)
- net USB_SSTXM_DN4: now reaches U1.27 (USB_SSTXM_DN4)
- net USB_SSRXP_DN4: now reaches U1.29 (USB_SSRXP_DN4)
- net USB_SSTXP_DN1: now reaches U1.3 (USB_SSTXP_DN1)
- net USB_SSRXM_DN4: now reaches U1.30 (USB_SSRXM_DN4)
- net USB_SSTXM_DN1: now reaches U1.4 (USB_SSTXM_DN1)
- net at U1.40 (FULLPWRMGMTz/SMBA1/SS_UP): now also R9.2
- net at U1.41 (PWRCTL_POL): now also R10.2
- net at U1.42 (GANGED/SMBA2/HS_UP): now also R8.2
- net at U1.45 (AUTOENz/HS_SUSPEND): now also R7.2
- net at U1.48 (USB_VBUS): now also R12.2, R13.2
- net at U1.49 (TEST): now also R6.2
- net at U1.50 (GRSTz): now also SW2.2 (B)
- net USB_DP_UP: now reaches U1.53 (USB_DP_UP)
- net USB_DM_UP: now reaches U1.54 (USB_DM_UP)
- net USB_SSTXP_UP: now reaches U1.55 (USB_SSTXP_UP)
- net USB_SSTXM_UP: now reaches U1.56 (USB_SSTXM_UP)
- net USB_SSRXP_UP: now reaches U1.58 (USB_SSRXP_UP)
- net USB_SSRXM_UP: now reaches U1.59 (USB_SSRXM_UP)
- net USB_SSRXP_DN1: now reaches U1.6 (USB_SSRXP_DN1)
- net at U1.64 (USB_R1): now also R11.2
- net USB_SSRXM_DN1: now reaches U1.7 (USB_SSRXM_DN1)
- net USB_DP_DN2: now reaches U1.9 (USB_DP_DN2)
- net VDD renamed +1V1
- net +1V1: now also C10.1, C11.1, C12.1, C13.1, C14.1, C15.1, C5.1, C8.1, C9.1, L1.2, U5.4 (FB)
- net XI renamed USB XI
- net XO renamed USB XO
- new net: L2.1, U4.8 (LX)
- new net: C4.1, U4.3 (VCC)
- new net: L1.1, U5.5 (SW)
- new net: R15.2, R16.1, U6.1 (DO)
- new net EEPROM SCL/SMBCLK: U2.6 (SCL)
- new net EEPROM SDA/SMBDAT: U2.5 (SDA)
- new net VCC: R12.1, U4.1 (VIN), U4.2 (EN/UVLO)
- no-connect marks 0 -> 1
Other:
- note added: "1v1 Supply"
- note added: "3v3 Supply"
- note added: "4.7k/5% ->"
- note added: "EEPROM FT4232"
- note added: "Power Supply Coupling"
- note added: "USB EEPROM"
- note added: "XTAL FT4232"
- note added: "XTAL TUSB8041"
- note removed: "EEPROM Stuff"
- note removed: "XTAL"
- moved on the sheet: J5, R2, R3, R4, R5, U2, U3

Commit message: push
Connections:
- net +3.3V: now also U3.50 (VREGIN)
- net VCORE: now also U3.49 (VREGOUT)
Changed lines of the file:
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@@
 	(wire
 		(pts
+			(xy 245.11 38.1) (xy 237.49 38.1)
+		)
+		(stroke
+			(width 0)
+			(type default)
+		)
+	)
+	(wire
+		(pts
 			(xy 109.22 229.87) (xy 114.3 229.87)
 		)
@@
 	(wire
 		(pts
+			(xy 237.49 43.18) (xy 245.11 43.18)
+		)
+		(stroke
+			(width 0)
+			(type default)
+		)
+	)
+	(wire
+		(pts
 			(xy 218.44 182.88) (xy 218.44 195.58)
 		)
@@
 	(wire
 		(pts
+			(xy 237.49 38.1) (xy 237.49 34.29)
+		)
+		(stroke
+			(width 0)
+			(type default)
+		)
+	)
+	(wire
+		(pts
 			(xy 275.59 139.7) (xy 275.59 142.24)
 		)
@@
 		)
 	)
+	(label "VCORE"
+		(at 237.49 43.18 180)
+		(effects
+			(font
+				(size 1.27 1.27)
+			)
+			(justify right bottom)
+		)
+	)
 	(label "SMBUSz{slash}SS_SUSPEND"
 		(at 381 29.21 0)
@@
 					(unit 1)
 				)
+			)
+		)
+	)
+	(symbol
+		(lib_id "power:+3.3V")
+		(at 237.49 34.29 0)
+		(unit 1)
+		(exclude_from_sim no)
+		(in_bom yes)
+		(on_board yes)
+		(dnp no)
+		(fields_autoplaced yes)
+		(property "Reference" "#PWR036"
+			(at 237.49 38.1 0)
+			(effects
+				(font
+					(size 1.27 1.27)
+				)
+				(hide yes)
+			)
+		)
+		(property "Value" "+3.3V"
+			(at 237.49 29.21 0)
+			(effects
+				(font
+					(size 1.27 1.27)
+				)
+			)
+		)
+		(property "Footprint" ""
+			(at 237.49 34.29 0)
+			(effects
+				(font
+					(size 1.27 1.27)
+				)
+				(hide yes)
+			)
+		)
+		(property "Datasheet" ""
+			(at 237.49 34.29 0)
+			(effects
+				(font
+					(size 1.27 1.27)
+				)
+				(hide yes)
+			)
+		)
+		(property "Description" "Power symbol creates a global label with name \"+3.3V\""
+			(at 237.49 34.29 0)
+			(effects
+				(font
+					(size 1.27 1.27)
+				)
+				(hide yes)
+			)
+		)
+		(pin "1"
+		)
+		(instances
+			(project "USB_3.0_Hub"
+				(path "/16fcb470-73b2-4b1c-a0c0-bdafed6619f6"
+					(reference "#PWR036")
+					(unit 1)
+				)
